File: cb-1/cb-1.kicad_sch (KiCad schematic)
At the start: 119 parts, among them CN0 Barrel_Jack, CN2 Mini-DIN-8, CN3 Cart_connector, CN4 LCD_Connector, Q9 Q_NPN_BCE, SW1 SW_SPST, SW10 3, SW11 6, SW12 9, SW13 C, SW14 2, SW15 5, SW16 8, SW17 ., SW18 1, SW19 4, SW2 RIGHT, SW20 7, SW21 0, SW3 UP, SW4 DOWN, SW5 LEFT, SW6 ADVICE, SW7 DC, SW8 M/B, SW9 OK, U1 AMS1117-5.0, U10 74HC373, U2 Reset IC, U3 74HC04, U4 74HC138, U5 uPD78213, U6 74LS32, U7 4075, U8 27C040, U9 CXK58257AP

Commit message: Add decoupling capacitors
Parts:
- added C12, C20, C21, C22, C23, C24, C30, C31: C, Capacitor_THT:C_Disc_D4.3mm_W1.9mm_P5.00mm, symbol Device:C
- added R10: R, Resistor_THT:R_Axial_DIN0207_L6.3mm_D2.5mm_P10.16mm_Horizontal, symbol Device:R
- renumbered C3 to C14
Connections:
- net +5V: now also C20.1, C21.1, C22.1, C23.2, C24.1, C30.2, R10.2
- net GND: now also C12.2, C20.2, C21.2, C22.2, C23.1, C24.2, C30.1, C31.1
- net SCK: now also R10.1
- net VMEM: now also C31.2
- net ~{MISO}: now also C12.1
Other:
- moved on the sheet: BT1, C28, C4, C5, C9, CN0, CN5, D2, D6, D7, F1, I1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
